File: mini-MIDI-hub.brd (EAGLE design)
At the start: 140.8 x 19.1 mm, 59 parts, among them IC1 6N138, IC2 4050D, IC3 REG1117, IC5 REG1117, X1 DIN5PIN, X2 DIN5PIN, X3 DIN5PIN, X4 DIN5PIN, X5 DIN5PIN, X6 DIN5PIN

Commit message: updates
Parts:
- removed C6: (no value), rcl:C0805
- removed R3: (no value), rcl:R0805
- removed U$1: PIC16F1825SO14, jasons_stuff:SO14
- added C11: (no value), rcl:E2-4
- added IC6: (no value), microbuilder:SOIC-4
- added R19: (no value), rcl:R0805
- C4, C9: device rcl:E2-4 -> rcl:C0805
- C8: device rcl:C0805 -> rcl:E2-4
- IC2: value 4050D -> PIC16F1825SO14; device 40xx:SO16 -> jasons_stuff:SO14
- IC3: value REG1117 -> 4050D; device burr-brown:SOT223 -> 40xx:SO16
- IC4: value (none) -> REG1117; device microbuilder:SOIC-4 -> burr-brown:SOT223
- moved R4 81.2 mm to (108.0, 16.5), turned to 270 degrees
- moved R5 81.1 mm to (114.3, 16.5)
- moved R10 78.6 mm to (8.38, 3.68)
- moved C2 76.4 mm to (19.1, 10.2), turned to 90 degrees
- moved R12 72.4 mm to (34.3, 3.56), turned to 270 degrees
- moved R14 69.3 mm to (54.0, 3.81), turned to 270 degrees
- moved R7 67.9 mm to (120.7, 16.5)
- moved R13 67.2 mm to (47.6, 3.81)
- moved R6 67.2 mm to (114.3, 11.8)
- moved R11 65.5 mm to (27.8, 3.56), turned to 90 degrees
- moved C3 60.3 mm to (33.0, 17.1), turned to 180 degrees
- moved R16 59.1 mm to (73.7, 3.81)
- moved R15 51.7 mm to (67.3, 3.81), turned to 90 degrees
- moved R8 51.7 mm to (118.5, 10.8), turned to 180 degrees
- moved R9 49.7 mm to (122.9, 10.8), turned to 0 degrees
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Connections:
- net 3V3: now also C3.2, C5.+, C7.1, IC2.1, IC4.2, R2.1; no longer C10.1, C8.2, C9.+, IC5.2, R1.1, U$1.1
- net 5V: now also C10.1, C4.1, C8.+, IC3.1, IC4.3, IC5.2, R11.2, R13.2, R15.2, R19.2, R5.2, R7.2; no longer C1.1, C2.1, C5.+, IC2.1, IC3.2, IC5.3, R10.2, R12.2, R20.2, R22.2, R6.2, R8.2
- net GND: now also C1.1, C11.-, C2.1, C3.1, C4.2, C7.2, C8.-, C9.2, IC2.14, IC3.8, IC4.1, IC6.-, R1.1, R6.1, R8.1, R9.1; no longer C1.2, C2.2, C3.2, C4.-, C6.1, C7.1, C8.1, C9.-, IC2.8, IC3.1, IC4.-, R13.1, R14.1, R15.1, R3.1, U$1.14
- net IN1: now also IC2.11; no longer U$1.11
- net IN2: now also IC2.8; no longer U$1.8
- net LEDA: now also IC2.13; no longer U$1.13
- net LEDB: now also IC2.12; no longer U$1.12
- net LEDC: now also IC2.7; no longer U$1.7
- net N$1: now also R12.2; no longer R5.2
- net N$10: now also IC3.10, R18.1; no longer IC2.10, R11.1
- net N$11: now also IC3.6, R14.1; no longer IC2.6, R7.1
- net N$12: now also IC3.2, R12.1; no longer IC2.2, R5.1
- net N$13: now also R8.2; no longer R15.2
- net N$14: now also R11.1; no longer R4.1
- net N$15: now also R13.1; no longer R6.1
- net N$16: now also R15.1; no longer R8.1
- net N$17: now also R17.1; no longer R10.1
- net N$18: now also R19.1; no longer R12.1
- net N$19: now also R21.1; no longer R17.1
- net N$2: now also R14.2; no longer R7.2
- net N$20: now also R10.1; no longer R2.1
- net N$21: now also R10.2; no longer R2.2
- net N$22: now also R1.2; no longer R3.2
- net N$23: now also R9.2; no longer R14.2
- net N$25: now also R6.2; no longer R13.2
- net N$27: now also IC6.~1; no longer IC4.~1
- net N$28: now also IC6.~2; no longer IC4.~2
- net N$29: now also C1.2, IC2.2; no longer C6.2, U$1.2
- net N$3: now also R16.2; no longer R9.2
- net N$30: now also C2.2, IC2.3; no longer C7.2, U$1.3
- net N$31: now also R4.1; no longer R20.1
- net N$32: now also R5.1; no longer R21.1
- net N$33: now also R7.1; no longer R22.1
- net N$36: now also IC2.4; no longer U$1.4
- net N$4: now also R18.2; no longer R11.2
- net N$5: now also R20.2; no longer R18.2
- net N$6: now also R22.2; no longer R16.2
- net N$7: now also IC3.15, R22.1; no longer IC2.15, R16.1
- net N$8: now also IC3.4, R16.1; no longer IC2.4, R9.1
- net N$9: now also IC3.12, R20.1; no longer IC2.12, R18.1
- net RX: now also IC2.5, R2.2; no longer R1.2, U$1.5
- net SCL: now also IC2.10; no longer U$1.10
- net SDA: now also IC2.9; no longer U$1.9
- net TX: now also IC2.6, IC3.11, IC3.14, IC3.3, IC3.5, IC3.7, IC3.9; no longer IC2.11, IC2.14, IC2.3, IC2.5, IC2.7, IC2.9, U$1.6
- net VIN: now also C11.+, C9.1, IC5.3, IC6.+; no longer C3.1, C4.+, IC3.3, IC4.+
Routing:
- net GND: track 73.0 -> 71.5 mm
- net LEDB: track 80.9 -> 81.8 mm
- net 5V: track 219.2 -> 218.7 mm, vias 12 -> 11
Other:
- board size 140.8 x 19.1 mm -> 140.9 x 19.3 mm
- board text added: "mini midi hub"
- board text added: "rev 1"

Commit message: tweakz
Parts:
- renumbered J1 to ICSP
Changed lines of the file:
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@@
 <wire x1="140.843" y1="1.27" x2="140.843" y2="7.366" width="0.4064" layer="20"/>
 <wire x1="140.843" y1="7.366" x2="139.7" y2="8.382" width="0.4064" layer="20" curve="90"/>
-<text x="129.1082" y="6.4262" size="1.27" layer="25" font="vector">hotchk155</text>
+<text x="72.1106" y="18.6944" size="1.27" layer="25" font="vector" rot="R180">hotchk155</text>
 <text x="57.404" y="7.5184" size="1.778" layer="25" font="vector">mini midi hub</text>
 <text x="57.4802" y="7.4422" size="1.778" layer="25" font="vector">mini midi hub</text>
@@
 <attribute name="NAME" x="37.084" y="8.5598" size="1.27" layer="25"/>
 </element>
-<element name="J1" library="tag-connect" package="TC2030-MCP-NL" value="" x="39.878" y="16.637" smashed="yes" rot="MR270">
-<attribute name="NAME" x="38.608" y="17.272" size="1.27" layer="26" rot="MR270"/>
+<element name="ICSP" library="tag-connect" package="TC2030-MCP-NL" value="" x="39.878" y="16.637" smashed="yes" rot="MR270">
+<attribute name="NAME" x="37.719" y="10.16" size="1.27" layer="26" rot="MR180"/>
 </element>
 <element name="R6" library="rcl" package="R0805" value="" x="114.3" y="11.811" smashed="yes" rot="R90">
@@
 <attribute name="MF" value="" x="69.1134" y="13.1572" size="1.778" layer="27" rot="R270" display="off"/>
 <attribute name="OC_FARNELL" value="1097566" x="69.1134" y="13.1572" size="1.778" layer="27" rot="R270" display="off"/>
-<attribute name="NAME" x="66.9544" y="16.51" size="1.27" layer="25" ratio="10"/>
+<attribute name="NAME" x="74.9046" y="11.6332" size="1.27" layer="25" ratio="10" rot="R90"/>
 </element>
 <element name="C5" library="rcl" package="E2-4" value="" x="59.69" y="16.51" smashed="yes">
@@
 <wire x1="18.984" y1="9.144" x2="19.05" y2="9.21" width="0.3048" layer="1"/>
 <contactref element="IC2" pad="14"/>
-<contactref element="J1" pad="3"/>
+<contactref element="ICSP" pad="3"/>
 <contactref element="C3" pad="1"/>
 <wire x1="35.62" y1="15.367" x2="35.62" y2="16.704" width="0.3048" layer="1"/>
@@
 <signal name="N$36">
 <contactref element="IC2" pad="4"/>
-<contactref element="J1" pad="1"/>
+<contactref element="ICSP" pad="1"/>
 <wire x1="40.513" y1="15.367" x2="42.037" y2="15.367" width="0.3048" layer="16"/>
 <via x="33.02" y="15.367" extent="1-16" drill="0.6"/>
@@
 <contactref element="LED2" pad="A"/>
 <contactref element="IC2" pad="13"/>
-<contactref element="J1" pad="4"/>
+<contactref element="ICSP" pad="4"/>
 <wire x1="35.62" y1="14.097" x2="37.719" y2="14.097" width="0.3048" layer="1"/>
 <via x="37.719" y="14.097" extent="1-16" drill="0.6"/>
@@
 <contactref element="LED3" pad="A"/>
 <contactref element="IC2" pad="12"/>
-<contactref element="J1" pad="5"/>
+<contactref element="ICSP" pad="5"/>
 <wire x1="35.62" y1="12.827" x2="42.037" y2="12.827" width="0.3048" layer="1"/>
 <via x="42.037" y="12.827" extent="1-16" drill="0.6"/>
@@
 </signal>
 <signal name="VDD">
-<contactref element="J1" pad="2"/>
+<contactref element="ICSP" pad="2"/>
 </signal>
 <signal name="N$34">

Commit message: tweaks
Parts:
- added R24, R25: (no value), rcl:R0805
- moved ICSP 4.74 mm to (44.6, 16.0), turned to 0 degrees
Connections:
- net 3V3: now also R24.1, R25.1
- net SCL: now also R25.2
- net SDA: now also R24.2
Routing:
- net 3V3: track 70.8 -> 87.4 mm, vias 1 -> 2
- net LEDB: track 81.8 -> 96.4 mm
- net LEDA: track 88.8 -> 96.1 mm, vias 4 -> 3
- net IN1: track 47.6 -> 52.9 mm
- net SCL: track 35.7 -> 39.5 mm
- net TX: track 62.0 -> 58.3 mm
- net SDA: track 38.2 -> 41.7 mm
- net N$36: track 15.9 -> 19.1 mm
- net 5V: track 218.7 -> 217.8 mm
- net IN2: track 48.7 -> 48.2 mm
- net GND: vias 10 -> 12
- added copper zone on layer 1, net GND

Commit message: pcb rev 1
Parts:
- turned U$2 to 0 degrees
- turned U$3 to 0 degrees
- turned U$4 to 0 degrees
Connections:
- removed net N$33: R7.1, U$4.K
- new net N$26: R4.1, U$2.A
- net N$31: now also R5.1, U$3.A; no longer R4.1, U$2.K
- net N$32: now also R7.1, U$4.A; no longer R5.1, U$3.K
- net N$34: now also U$2.K, U$3.K, U$4.K; no longer U$2.A, U$3.A, U$4.A
Routing:
- net N$26: track 0.00 -> 2.23 mm
- net N$33: track 2.04 -> 0.00 mm
- net N$34: track 25.7 -> 24.2 mm
Other:
- outline, holes or cut-outs redrawn
Changed lines of the file:
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@@
 <board>
 <plain>
-<wire x1="139.7" y1="8.382" x2="127" y2="8.382" width="0.4064" layer="20"/>
-<wire x1="127" y1="8.382" x2="126.492" y2="8.89" width="0.4064" layer="20" curve="-90"/>
-<wire x1="126.492" y1="8.89" x2="126.492" y2="17.78" width="0.4064" layer="20"/>
-<wire x1="126.492" y1="17.78" x2="124.4854" y2="19.304" width="0.4064" layer="20" curve="90"/>
-<wire x1="124.4854" y1="19.304" x2="1.0922" y2="19.304" width="0.4064" layer="20"/>
+<wire x1="139.7" y1="8.382" x2="127.508" y2="8.382" width="0.4064" layer="20"/>
+<wire x1="127.508" y1="8.382" x2="126.746" y2="8.89" width="0.4064" layer="20" curve="-90"/>
+<wire x1="126.746" y1="8.89" x2="126.746" y2="18.542" width="0.4064" layer="20"/>
+<wire x1="126.746" y1="18.542" x2="126.0094" y2="19.304" width="0.4064" layer="20" curve="90"/>
+<wire x1="126.0094" y1="19.304" x2="1.0922" y2="19.304" width="0.4064" layer="20"/>
 <wire x1="1.0922" y1="19.304" x2="0" y2="17.907" width="0.4064" layer="20" curve="90"/>
 <wire x1="0" y1="17.907" x2="0" y2="1.0668" width="0.4064" layer="20"/>
@@
 <attribute name="VALUE" x="97.8408" y="17.145" size="1.27" layer="27" rot="R270"/>
 </element>
-<element name="U$2" library="jason_eagle6" package="LED5MM_EDGE" value="LED5MM_EDGE" x="111.125" y="17.78" smashed="yes" rot="R180"/>
-<element name="U$3" library="jason_eagle6" package="LED5MM_EDGE" value="LED5MM_EDGE" x="117.475" y="17.78" smashed="yes" rot="R180"/>
-<element name="U$4" library="jason_eagle6" package="LED5MM_EDGE" value="LED5MM_EDGE" x="123.825" y="17.78" smashed="yes" rot="R180"/>
+<element name="U$2" library="jason_eagle6" package="LED5MM_EDGE" value="LED5MM_EDGE" x="111.125" y="17.78" smashed="yes"/>
+<element name="U$3" library="jason_eagle6" package="LED5MM_EDGE" value="LED5MM_EDGE" x="117.475" y="17.78" smashed="yes"/>
+<element name="U$4" library="jason_eagle6" package="LED5MM_EDGE" value="LED5MM_EDGE" x="123.825" y="17.78" smashed="yes"/>
 <element name="R25" library="rcl" package="R0805" value="" x="40.0558" y="11.176" smashed="yes" rot="R180">
 <attribute name="NAME" x="38.5572" y="12.192" size="1.27" layer="25"/>
@@
 <signal name="N$34">
 <contactref element="T1" pad="C"/>
-<contactref element="U$2" pad="A"/>
-<contactref element="U$3" pad="A"/>
-<contactref element="U$4" pad="A"/>
 <wire x1="104.8336" y1="16.4846" x2="106.1212" y2="16.4846" width="0.3048" layer="1"/>
 <via x="106.1212" y="16.4846" extent="1-16" drill="0.7"/>
-<wire x1="106.1212" y1="16.4846" x2="110.49" y2="16.4846" width="0.3048" layer="16"/>
-<wire x1="110.49" y1="16.4846" x2="116.84" y2="16.4846" width="0.3048" layer="16"/>
-<wire x1="116.84" y1="16.4846" x2="123.1646" y2="16.4846" width="0.3048" layer="16"/>
-<wire x1="123.1646" y1="16.4846" x2="124.46" y2="17.78" width="0.3048" layer="16"/>
-<wire x1="124.46" y1="17.78" x2="125.095" y2="17.78" width="0.3048" layer="16"/>
-<wire x1="118.745" y1="17.78" x2="118.11" y2="17.78" width="0.3048" layer="16"/>
-<wire x1="118.11" y1="17.78" x2="116.84" y2="16.51" width="0.3048" layer="16"/>
+<wire x1="106.1212" y1="16.4846" x2="112.395" y2="16.4846" width="0.3048" layer="16"/>
+<wire x1="112.395" y1="16.4846" x2="116.84" y2="16.4846" width="0.3048" layer="16"/>
+<wire x1="116.84" y1="16.4846" x2="118.7196" y2="16.4846" width="0.3048" layer="16"/>
+<wire x1="118.7196" y1="16.4846" x2="125.095" y2="16.4846" width="0.3048" layer="16"/>
 <wire x1="116.84" y1="16.51" x2="116.84" y2="16.4846" width="0.3048" layer="16"/>
-<wire x1="112.395" y1="17.78" x2="111.7854" y2="17.78" width="0.3048" layer="16"/>
-<wire x1="111.7854" y1="17.78" x2="110.49" y2="16.4846" width="0.3048" layer="16"/>
+<contactref element="U$2" pad="K"/>
+<contactref element="U$3" pad="K"/>
+<contactref element="U$4" pad="K"/>
+<wire x1="118.745" y1="17.78" x2="118.7196" y2="17.78" width="0.3048" layer="16"/>
+<wire x1="118.7196" y1="17.78" x2="118.7196" y2="16.4846" width="0.3048" layer="16"/>
+<wire x1="125.095" y1="17.78" x2="125.095" y2="16.4846" width="0.3048" layer="16"/>
+<wire x1="112.395" y1="17.78" x2="112.395" y2="16.4846" width="0.3048" layer="16"/>
 </signal>
 <signal name="N$39">
@@
 <wire x1="102.6082" y1="17.46" x2="102.6336" y2="17.4346" width="0.3048" layer="1"/>
 </signal>
+<signal name="N$26">
+<contactref element="U$2" pad="A"/>
+<contactref element="R4" pad="1"/>
+<wire x1="109.855" y1="17.78" x2="107.95" y2="17.78" width="0.3048" layer="1"/>
+<wire x1="107.95" y1="17.78" x2="107.95" y2="17.46" width="0.3048" layer="1"/>
+</signal>
 <signal name="N$31">
-<contactref element="R4" pad="1"/>
-<contactref element="U$2" pad="K"/>
-<wire x1="109.855" y1="17.78" x2="108.27" y2="17.78" width="0.3048" layer="1"/>
-<wire x1="108.27" y1="17.78" x2="107.95" y2="17.46" width="0.3048" layer="1"/>
+<contactref element="U$3" pad="A"/>
+<contactref element="R5" pad="1"/>
+<wire x1="116.205" y1="17.78" x2="114.3" y2="17.78" width="0.3048" layer="1"/>
+<wire x1="114.3" y1="17.78" x2="114.3" y2="17.46" width="0.3048" layer="1"/>
 </signal>
 <signal name="N$32">
-<contactref element="R5" pad="1"/>
-<contactref element="U$3" pad="K"/>
-<wire x1="116.205" y1="17.78" x2="114.62" y2="17.78" width="0.3048" layer="1"/>
-<wire x1="114.62" y1="17.78" x2="114.3" y2="17.46" width="0.3048" layer="1"/>
-</signal>
-<signal name="N$33">
+<contactref element="U$4" pad="A"/>
 <contactref element="R7" pad="1"/>
-<contactref element="U$4" pad="K"/>
-<wire x1="122.555" y1="17.78" x2="120.97" y2="17.78" width="0.3048" layer="1"/>
-<wire x1="120.97" y1="17.78" x2="120.65" y2="17.46" width="0.3048" layer="1"/>
+<wire x1="122.555" y1="17.78" x2="120.65" y2="17.78" width="0.3048" layer="1"/>
+<wire x1="120.65" y1="17.78" x2="120.65" y2="17.46" width="0.3048" layer="1"/>
 </signal>
 </signals>
