File: mini-MIDI-hub.sch (EAGLE design)
At the start: 59 parts, among them IC1 6N138, IC2 4050D, IC3 REG1117, IC5 REG1117, X1 DIN5PIN, X2 DIN5PIN, X3 DIN5PIN, X4 DIN5PIN, X5 DIN5PIN, X6 DIN5PIN

Commit message: updates
Parts:
- removed C6: (no value), rcl:C-EUC0805
- removed R3: (no value), rcl:R-EU_R0805
- removed U$1: PIC16F1825SO14, jasons_stuff:PIC16F1825SO14
- added C11: (no value), rcl:CPOL-EUE2-4
- added IC6: (no value), microbuilder:BRIDGERECTIFIER
- added R19: (no value), rcl:R-EU_R0805
- C4, C9: device rcl:CPOL-EUE2-4 -> rcl:C-EUC0805
- C8: device rcl:C-EUC0805 -> rcl:CPOL-EUE2-4
- IC2: value 4050D -> PIC16F1825SO14; device 40xx:4050D -> jasons_stuff:PIC16F1825SO14
- IC3: value REG1117 -> 4050D; device burr-brown:REG1117 -> 40xx:4050D
- IC4: value (none) -> REG1117; device microbuilder:BRIDGERECTIFIER -> burr-brown:REG1117
Connections:
- net 3V3: now also C3.2, C5.+, C7.1, IC2.VDD, IC4.VOUT, R2.1; no longer C10.1, C8.2, C9.+, IC5.VOUT, R1.1, U$1.VDD
- net 5V: now also C10.1, C4.1, C8.+, IC3P.VDD, IC4.VIN, IC5.VOUT, R11.2, R13.2, R15.2, R19.2, R5.2, R7.2; no longer C1.1, C2.1, C5.+, IC2P.VDD, IC3.VOUT, IC5.VIN, R10.2, R12.2, R20.2, R22.2, R6.2, R8.2
- net GND: now also C1.1, C11.-, C2.1, C3.1, C4.2, C7.2, C8.-, C9.2, IC2.VSS, IC3P.VSS, IC4.GND, IC6.-, R1.1, R6.1, R8.1, R9.1; no longer C1.2, C2.2, C3.2, C4.-, C6.1, C7.1, C8.1, C9.-, IC2P.VSS, IC3.GND, IC4.-, R13.1, R14.1, R15.1, R3.1, U$1.VSS
- net IN1: now also IC2.RA2/INT; no longer U$1.RA2/INT
- net IN2: now also IC2.RC2; no longer U$1.RC2
- net LEDA: now also IC2.RA0/ICSPDAT; no longer U$1.RA0/ICSPDAT
- net LEDB: now also IC2.RA1/ICPCLK; no longer U$1.RA1/ICPCLK
- net LEDC: now also IC2.RC3/SS#; no longer U$1.RC3/SS#
- net N$1: now also R12.2; no longer R5.2
- net N$10: now also IC3D.O, R18.1; no longer IC2D.O, R11.1
- net N$11: now also IC3C.O, R14.1; no longer IC2C.O, R7.1
- net N$12: now also IC3A.O, R12.1; no longer IC2A.O, R5.1
- net N$13: now also R8.2; no longer R15.2
- net N$14: now also R11.1; no longer R4.1
- net N$15: now also R13.1; no longer R6.1
- net N$16: now also R15.1; no longer R8.1
- net N$17: now also R17.1; no longer R10.1
- net N$18: now also R19.1; no longer R12.1
- net N$19: now also R21.1; no longer R17.1
- net N$2: now also R14.2; no longer R7.2
- net N$20: now also R10.1; no longer R2.1
- net N$21: now also R10.2; no longer R2.2
- net N$22: now also R1.2; no longer R3.2
- net N$23: now also R9.2; no longer R14.2
- net N$25: now also R6.2; no longer R13.2
- net N$27: now also IC6.AC1; no longer IC4.AC1
- net N$28: now also IC6.AC2; no longer IC4.AC2
- net N$29: now also C1.2, IC2.RA5; no longer C6.2, U$1.RA5
- net N$3: now also R16.2; no longer R9.2
- net N$30: now also C2.2, IC2.RA4/SDO; no longer C7.2, U$1.RA4/SDO
- net N$31: now also R4.1; no longer R20.1
- net N$32: now also R5.1; no longer R21.1
- net N$33: now also R7.1; no longer R22.1
- net N$36: now also IC2.RA3/MCLR#/VPP; no longer U$1.RA3/MCLR#/VPP
- net N$4: now also R18.2; no longer R11.2
- net N$5: now also R20.2; no longer R18.2
- net N$6: now also R22.2; no longer R16.2
- net N$7: now also IC3F.O, R22.1; no longer IC2F.O, R16.1
- net N$8: now also IC3B.O, R16.1; no longer IC2B.O, R9.1
- net N$9: now also IC3E.O, R20.1; no longer IC2E.O, R18.1
- net RX: now also IC2.RC5/RX, R2.2; no longer R1.2, U$1.RC5/RX
- net SCL: now also IC2.RCO/SCL/SCK; no longer U$1.RCO/SCL/SCK
- net SDA: now also IC2.RC1/SDA/SDI; no longer U$1.RC1/SDA/SDI
- net TX: now also IC2.RC4/TX, IC3A.I, IC3B.I, IC3C.I, IC3D.I, IC3E.I, IC3F.I; no longer IC2A.I, IC2B.I, IC2C.I, IC2D.I, IC2E.I, IC2F.I, U$1.RC4/TX
- net VIN: now also C11.+, C9.1, IC5.VIN, IC6.+; no longer C3.1, C4.+, IC3.VIN, IC4.+
Other:
- moved on the sheet: C1, C10, C2, C3, C5, C7, IC5, R1, R10, R11, R12, R13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

Commit message: tweakz
Parts:
- renumbered J1 to ICSP
Changed lines of the file:
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@@
 <part name="GND1" library="supply1" deviceset="GND" device=""/>
 <part name="IC2" library="jasons_stuff" deviceset="PIC16F1825" device="SO14"/>
-<part name="J1" library="tag-connect" deviceset="TC2030" device="-MCP-NL"/>
+<part name="ICSP" library="tag-connect" deviceset="TC2030" device="-MCP-NL"/>
 <part name="GND2" library="supply1" deviceset="GND" device=""/>
 <part name="GND3" library="supply1" deviceset="GND" device=""/>
@@
 <instance part="GND1" gate="1" x="317.5" y="33.02"/>
 <instance part="IC2" gate="G$1" x="360.68" y="38.1"/>
-<instance part="J1" gate="G$1" x="414.02" y="43.18"/>
+<instance part="ICSP" gate="G$1" x="414.02" y="43.18"/>
 <instance part="GND2" gate="1" x="15.24" y="33.02"/>
 <instance part="GND3" gate="1" x="22.86" y="33.02"/>
@@
 <segment>
 <pinref part="IC2" gate="G$1" pin="VSS"/>
-<pinref part="J1" gate="G$1" pin="VSS(GND)"/>
+<pinref part="ICSP" gate="G$1" pin="VSS(GND)"/>
 <wire x1="383.54" y1="45.72" x2="386.08" y2="45.72" width="0.1524" layer="91"/>
 <pinref part="C3" gate="G$1" pin="1"/>
@@
 <wire x1="337.82" y1="53.34" x2="398.78" y2="53.34" width="0.1524" layer="91"/>
 <wire x1="398.78" y1="53.34" x2="398.78" y2="50.8" width="0.1524" layer="91"/>
-<pinref part="J1" gate="G$1" pin="VPP/MCLR"/>
+<pinref part="ICSP" gate="G$1" pin="VPP/MCLR"/>
 <wire x1="401.32" y1="50.8" x2="398.78" y2="50.8" width="0.1524" layer="91"/>
 </segment>
@@
 <segment>
 <pinref part="IC2" gate="G$1" pin="RA0/ICSPDAT"/>
-<pinref part="J1" gate="G$1" pin="ICSP_DAT/PGD"/>
+<pinref part="ICSP" gate="G$1" pin="ICSP_DAT/PGD"/>
 <wire x1="383.54" y1="43.18" x2="388.62" y2="43.18" width="0.1524" layer="91"/>
 <wire x1="388.62" y1="43.18" x2="401.32" y2="43.18" width="0.1524" layer="91"/>
@@
 <segment>
 <pinref part="IC2" gate="G$1" pin="RA1/ICPCLK"/>
-<pinref part="J1" gate="G$1" pin="ICSP_CLK/PGC"/>
+<pinref part="ICSP" gate="G$1" pin="ICSP_CLK/PGC"/>
 <wire x1="383.54" y1="40.64" x2="391.16" y2="40.64" width="0.1524" layer="91"/>
 <wire x1="391.16" y1="40.64" x2="401.32" y2="40.64" width="0.1524" layer="91"/>

Commit message: tweaks
Parts:
- added R24, R25: (no value), rcl:R-EU_R0805
Connections:
- net 3V3: now also R24.1, R25.1
- net SCL: now also R25.2
- net SDA: now also R24.2
Changed lines of the file:
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@@
 <part name="U$3" library="jason_eagle6" deviceset="LED5MM_EDGE" device=""/>
 <part name="U$4" library="jason_eagle6" deviceset="LED5MM_EDGE" device=""/>
+<part name="R25" library="rcl" deviceset="R-EU_" device="R0805"/>
+<part name="R24" library="rcl" deviceset="R-EU_" device="R0805"/>
 </parts>
 <sheets>
@@
 <instance part="GND1" gate="1" x="317.5" y="33.02"/>
 <instance part="IC2" gate="G$1" x="360.68" y="38.1"/>
-<instance part="ICSP" gate="G$1" x="414.02" y="43.18"/>
+<instance part="ICSP" gate="G$1" x="419.1" y="43.18"/>
 <instance part="GND2" gate="1" x="15.24" y="33.02"/>
 <instance part="GND3" gate="1" x="22.86" y="33.02"/>
@@
 <instance part="U$3" gate="G$1" x="17.78" y="-2.54" rot="R270"/>
 <instance part="U$4" gate="G$1" x="22.86" y="-2.54" rot="R270"/>
+<instance part="R25" gate="G$1" x="393.7" y="63.5" rot="R270"/>
+<instance part="R24" gate="G$1" x="396.24" y="63.5" rot="R270"/>
 </instances>
 <busses>
@@
 <wire x1="383.54" y1="45.72" x2="386.08" y2="45.72" width="0.1524" layer="91"/>
 <pinref part="C3" gate="G$1" pin="1"/>
-<wire x1="386.08" y1="45.72" x2="401.32" y2="45.72" width="0.1524" layer="91"/>
+<wire x1="386.08" y1="45.72" x2="406.4" y2="45.72" width="0.1524" layer="91"/>
 <wire x1="365.76" y1="58.42" x2="386.08" y2="58.42" width="0.1524" layer="91"/>
 <wire x1="386.08" y1="58.42" x2="386.08" y2="45.72" width="0.1524" layer="91"/>
@@
 <pinref part="IC2" gate="G$1" pin="RA3/MCLR#/VPP"/>
 <wire x1="340.36" y1="38.1" x2="337.82" y2="38.1" width="0.1524" layer="91"/>
-<wire x1="337.82" y1="38.1" x2="337.82" y2="53.34" width="0.1524" layer="91"/>
-<wire x1="337.82" y1="53.34" x2="398.78" y2="53.34" width="0.1524" layer="91"/>
-<wire x1="398.78" y1="53.34" x2="398.78" y2="50.8" width="0.1524" layer="91"/>
+<wire x1="337.82" y1="38.1" x2="337.82" y2="50.8" width="0.1524" layer="91"/>
+<wire x1="337.82" y1="50.8" x2="406.4" y2="50.8" width="0.1524" layer="91"/>
 <pinref part="ICSP" gate="G$1" pin="VPP/MCLR"/>
-<wire x1="401.32" y1="50.8" x2="398.78" y2="50.8" width="0.1524" layer="91"/>
 </segment>
 </net>
@@
 <segment>
 <pinref part="IC2" gate="G$1" pin="RCO/SCL/SCK"/>
-<wire x1="383.54" y1="35.56" x2="388.62" y2="35.56" width="0.1524" layer="91"/>
-<label x="388.62" y="35.56" size="1.778" layer="95"/>
+<wire x1="383.54" y1="35.56" x2="393.7" y2="35.56" width="0.1524" layer="91"/>
+<label x="398.78" y="35.56" size="1.778" layer="95"/>
+<pinref part="R25" gate="G$1" pin="2"/>
+<wire x1="393.7" y1="35.56" x2="398.78" y2="35.56" width="0.1524" layer="91"/>
+<wire x1="393.7" y1="58.42" x2="393.7" y2="35.56" width="0.1524" layer="91"/>
+<junction x="393.7" y="35.56"/>
 </segment>
 <segment>
@@
 <segment>
 <pinref part="IC2" gate="G$1" pin="RC1/SDA/SDI"/>
-<wire x1="383.54" y1="33.02" x2="388.62" y2="33.02" width="0.1524" layer="91"/>
-<label x="388.62" y="33.02" size="1.778" layer="95"/>
+<wire x1="383.54" y1="33.02" x2="396.24" y2="33.02" width="0.1524" layer="91"/>
+<label x="398.78" y="33.02" size="1.778" layer="95"/>
+<pinref part="R24" gate="G$1" pin="2"/>
+<wire x1="396.24" y1="33.02" x2="398.78" y2="33.02" width="0.1524" layer="91"/>
+<wire x1="396.24" y1="58.42" x2="396.24" y2="33.02" width="0.1524" layer="91"/>
+<junction x="396.24" y="33.02"/>
 </segment>
 <segment>
@@
 <pinref part="ICSP" gate="G$1" pin="ICSP_DAT/PGD"/>
 <wire x1="383.54" y1="43.18" x2="388.62" y2="43.18" width="0.1524" layer="91"/>
-<wire x1="388.62" y1="43.18" x2="401.32" y2="43.18" width="0.1524" layer="91"/>
+<wire x1="388.62" y1="43.18" x2="406.4" y2="43.18" width="0.1524" layer="91"/>
 <wire x1="388.62" y1="43.18" x2="388.62" y2="58.42" width="0.1524" layer="91"/>
 <junction x="388.62" y="43.18"/>
@@
 <pinref part="ICSP" gate="G$1" pin="ICSP_CLK/PGC"/>
 <wire x1="383.54" y1="40.64" x2="391.16" y2="40.64" width="0.1524" layer="91"/>
-<wire x1="391.16" y1="40.64" x2="401.32" y2="40.64" width="0.1524" layer="91"/>
+<wire x1="391.16" y1="40.64" x2="406.4" y2="40.64" width="0.1524" layer="91"/>
 <wire x1="391.16" y1="40.64" x2="391.16" y2="58.42" width="0.1524" layer="91"/>
 <junction x="391.16" y="40.64"/>
@@
 <junction x="340.36" y="58.42"/>
 <label x="337.82" y="76.2" size="1.778" layer="95"/>
+<wire x1="340.36" y1="58.42" x2="340.36" y2="76.2" width="0.1524" layer="91"/>
 </segment>
 <segment>
@@
 <label x="228.6" y="116.84" size="1.778" layer="95"/>
 </segment>
-</net>
+<segment>
+<pinref part="R25" gate="G$1" pin="1"/>
+<wire x1="393.7" y1="68.58" x2="393.7" y2="71.12" width="0.1524" layer="91"/>
+<pinref part="R24" gate="G$1" pin="1"/>
+<wire x1="393.7" y1="71.12" x2="396.24" y2="71.12" width="0.1524" layer="91"/>
+<wire x1="396.24" y1="71.12" x2="396.24" y2="68.58" width="0.1524" layer="91"/>
+<wire x1="393.7" y1="71.12" x2="393.7" y2="78.74" width="0.1524" layer="91"/>
+<junction x="393.7" y="71.12"/>
+<label x="391.16" y="78.74" size="1.778" layer="95"/>
+</segment>
+</net>

Commit message: pcb rev 1
Other:
- moved on the sheet: C1, C2, C3, C4, IC1, IC3A, IC3B, IC3C, IC3D, IC3E, IC3F, IC3P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
